Commit message: added velocity smoother to help prevent spot from tipping over

File: spot_description_sim/sdf/model.sdf.xacro (robot description, xacro)
@@ -26,10 +26,6 @@
         <mass>1e-05</mass>
         <inertia>
-          <ixx>0.001</ixx>
-          <ixy>1e-06</ixy>
-          <ixz>1e-06</ixz>
-          <iyy>0.001</iyy>
-          <iyz>1e-06</iyz>
-          <izz>0.001</izz>
+          <ixx>1e-09</ixx><ixy>0</ixy><ixz>0</ixz>
+          <iyy>1e-09</iyy><iyz>0</iyz><izz>1e-09</izz>
         </inertia>
       </inertial>
@@ -130,4 +126,5 @@
     <link name="payload_mount_reference_frame">
       <pose>${payload_x} 0 ${payload_z} 0 0 0</pose>
+      <xacro:tiny_inertial/>
     </link>
     <joint name="payload_mount_reference_frame_joint" type="fixed">
@@ -245,4 +242,5 @@
     <link name="velodyne">
       <pose relative_to="velodyne_base_link">0 0 ${vlp16_optical_z} 0 0 0</pose>
+      <xacro:tiny_inertial/>
       <sensor name='gpu_lidar' type='gpu_lidar'>
         <pose>0 0 0 0 0 0</pose>
@@ -437,4 +435,5 @@
     <!-- ================= IMU ================= -->
     <link name="imu">
+      <xacro:tiny_inertial/>
       <sensor name="imu" type="imu">
         <always_on>1</always_on>
@@ -1107,9 +1106,11 @@
       <dimensions>3</dimensions>
     </plugin>
-    <xacro:macro name="pid_joint" params="joint p i d">
+    <xacro:macro name="pid_joint" params="joint p i d i_min:=-5.0 i_max:=5.0">
       <joint_name>${joint}</joint_name>
       <position_p_gain>${p}</position_p_gain>
       <position_i_gain>${i}</position_i_gain>
       <position_d_gain>${d}</position_d_gain>
+      <position_i_min>${i_min}</position_i_min>
+      <position_i_max>${i_max}</position_i_max>
     </xacro:macro>
     <plugin

Commit message: fixed SRDF error in RVIZ, added jointstate intializer for arm to be in stow state and updated world file to have correct ground plane

File: spot_description_sim/sdf/model.sdf.xacro (robot description, xacro)
@@ -804,5 +804,4 @@
       <axis>
         <xyz>0 1 0</xyz>
-        <initial_position>-3.1360</initial_position>
         <limit>
           <lower>-3.14159265358979311599</lower>
@@ -1106,6 +1105,7 @@
       <dimensions>3</dimensions>
     </plugin>
-    <xacro:macro name="pid_joint" params="joint p i d i_min:=-5.0 i_max:=5.0">
+    <xacro:macro name="pid_joint" params="joint p i d i_min:=-5.0 i_max:=5.0 init:=0.0">
       <joint_name>${joint}</joint_name>
+      <initial_position>${init}</initial_position>
       <position_p_gain>${p}</position_p_gain>
       <position_i_gain>${i}</position_i_gain>
@@ -1130,12 +1130,29 @@
       <xacro:pid_joint joint="rear_right_hip_y"  p="500" i="1" d="20"/>
       <xacro:pid_joint joint="rear_right_knee"   p="500" i="1" d="20"/>
-      <!-- Arm joints — arm0_shoulder_roll is fixed and excluded -->
-      <xacro:pid_joint joint="arm0_shoulder_yaw"   p="500" i="0" d="20"/>
-      <xacro:pid_joint joint="arm0_shoulder_pitch" p="500" i="0" d="20"/>
-      <xacro:pid_joint joint="arm0_elbow_pitch"    p="500" i="0" d="20"/>
-      <xacro:pid_joint joint="arm0_elbow_roll"     p="150" i="0" d="1"/>
-      <xacro:pid_joint joint="arm0_wrist_pitch"    p="150" i="0" d="2"/>
-      <xacro:pid_joint joint="arm0_wrist_roll"     p="80"  i="0" d="0.2"/>
-      <xacro:pid_joint joint="arm0_fingers"        p="30"  i="0" d="0.1"/>
+      <!-- Arm joints — arm0_shoulder_roll is fixed and excluded.
+           init values = STOW_CONFIG from sim_manipulation_driver.py, so the
+           controller's hold target matches the spawn pose set below. -->
+      <xacro:pid_joint joint="arm0_shoulder_yaw"   p="500" i="0" d="20"  init="-0.0011"/>
+      <xacro:pid_joint joint="arm0_shoulder_pitch" p="500" i="0" d="20"  init="-3.1360"/>
+      <xacro:pid_joint joint="arm0_elbow_pitch"    p="500" i="0" d="20"  init="3.1337"/>
+      <xacro:pid_joint joint="arm0_elbow_roll"     p="150" i="0" d="1"   init="1.5699"/>
+      <xacro:pid_joint joint="arm0_wrist_pitch"    p="150" i="0" d="2"   init="-0.0027"/>
+      <xacro:pid_joint joint="arm0_wrist_roll"     p="80"  i="0" d="0.2" init="-1.5684"/>
+      <xacro:pid_joint joint="arm0_fingers"        p="30"  i="0" d="0.1" init="0.0"/>
+    </plugin>
+    <!-- Kinematically teleport the arm to stow on the first physics step.
+         The JTC init targets above only make the PID *pull* toward stow
+         (a violent pi-radian swing at spawn that kicks the body over); this
+         plugin resets the joint states directly, so the arm is simply there.
+         Values = STOW_CONFIG (sim_manipulation_driver.py). -->
+    <plugin filename="JointStateInitializer"
+            name="spot_gazebo::JointStateInitializer">
+      <joint name="arm0_shoulder_yaw">-0.0011</joint>
+      <joint name="arm0_shoulder_pitch">-3.1360</joint>
+      <joint name="arm0_elbow_pitch">3.1337</joint>
+      <joint name="arm0_elbow_roll">1.5699</joint>
+      <joint name="arm0_wrist_pitch">-0.0027</joint>
+      <joint name="arm0_wrist_roll">-1.5684</joint>
+      <joint name="arm0_fingers">0.0</joint>
     </plugin>
   </model>

Commit message: updates to calibration world and test world

File: spot_description_sim/sdf/model.sdf.xacro (robot description, xacro)
@@ -427,5 +427,5 @@
                          x="${hand_rgb_x}" y="${hand_rgb_y}" z="${hand_rgb_z}"
                          pitch="${hand_rgb_pitch}"
-                         width="640" height="480" hfov="1.0472" far="15"/>
+                         width="1280" height="960" hfov="1.0472" far="15"/>
       <xacro:hand_camera name="tof" optical_frame="hand_depth_sensor"
                          x="${hand_tof_x}" y="${hand_tof_y}" z="${hand_tof_z}"
@@ -1133,10 +1133,10 @@
            init values = STOW_CONFIG from sim_manipulation_driver.py, so the
            controller's hold target matches the spawn pose set below. -->
-      <xacro:pid_joint joint="arm0_shoulder_yaw"   p="500" i="0" d="20"  init="-0.0011"/>
-      <xacro:pid_joint joint="arm0_shoulder_pitch" p="500" i="0" d="20"  init="-3.1360"/>
-      <xacro:pid_joint joint="arm0_elbow_pitch"    p="500" i="0" d="20"  init="3.1337"/>
-      <xacro:pid_joint joint="arm0_elbow_roll"     p="150" i="0" d="1"   init="1.5699"/>
-      <xacro:pid_joint joint="arm0_wrist_pitch"    p="150" i="0" d="2"   init="-0.0027"/>
-      <xacro:pid_joint joint="arm0_wrist_roll"     p="80"  i="0" d="0.2" init="-1.5684"/>
+      <xacro:pid_joint joint="arm0_shoulder_yaw"   p="1500" i="15" d="35" i_min="-50" i_max="50" init="-0.0011"/>
+      <xacro:pid_joint joint="arm0_shoulder_pitch" p="1500" i="15" d="35" i_min="-50" i_max="50" init="-3.1360"/>
+      <xacro:pid_joint joint="arm0_elbow_pitch"    p="1500" i="15" d="35" i_min="-50" i_max="50" init="3.1337"/>
+      <xacro:pid_joint joint="arm0_elbow_roll"     p="150" i="5" d="1"   init="1.5699"/>
+      <xacro:pid_joint joint="arm0_wrist_pitch"    p="150" i="8" d="2"   i_min="-15" i_max="15" init="-0.0027"/>
+      <xacro:pid_joint joint="arm0_wrist_roll"     p="80"  i="5" d="0.2" init="-1.5684"/>
       <xacro:pid_joint joint="arm0_fingers"        p="30"  i="0" d="0.1" init="0.0"/>
     </plugin>

Commit message: updates to controller

File: spot_description_sim/sdf/model.sdf.xacro (robot description, xacro)
@@ -1099,5 +1099,8 @@
       filename="ignition-gazebo-odometry-publisher-system"
       name="ignition::gazebo::systems::OdometryPublisher">
-      <odom_publish_frequency>10</odom_publish_frequency>
+      <!-- 100 Hz (was 10): at 10 Hz the odom stream was 20x sparser than the
+           200 Hz joint states, so TF odom->base updated in visible steps
+           relative to joint motion and EKF odom0 measurements were stale. -->
+      <odom_publish_frequency>100</odom_publish_frequency>
       <odom_topic>/model/spot/odometry</odom_topic>
       <odom_frame>odom</odom_frame>
@@ -1118,16 +1121,21 @@
       name="ignition::gazebo::systems::JointTrajectoryController">
       <topic>model/spot/joint_trajectory</topic>
-      <xacro:pid_joint joint="front_left_hip_x"  p="500" i="1" d="20"/>
-      <xacro:pid_joint joint="front_left_hip_y"  p="500" i="1" d="20"/>
-      <xacro:pid_joint joint="front_left_knee"   p="500" i="1" d="20"/>
-      <xacro:pid_joint joint="front_right_hip_x" p="500" i="1" d="20"/>
-      <xacro:pid_joint joint="front_right_hip_y" p="500" i="1" d="20"/>
-      <xacro:pid_joint joint="front_right_knee"  p="500" i="1" d="20"/>
-      <xacro:pid_joint joint="rear_left_hip_x"   p="500" i="1" d="20"/>
-      <xacro:pid_joint joint="rear_left_hip_y"   p="500" i="1" d="20"/>
-      <xacro:pid_joint joint="rear_left_knee"    p="500" i="1" d="20"/>
-      <xacro:pid_joint joint="rear_right_hip_x"  p="500" i="1" d="20"/>
-      <xacro:pid_joint joint="rear_right_hip_y"  p="500" i="1" d="20"/>
-      <xacro:pid_joint joint="rear_right_knee"   p="500" i="1" d="20"/>
+      <!-- Leg gains: p raised 500->900 and i 1->12 (clamp widened to +/-25 Nm)
+           so stance legs stop sagging under load — the robot is rear-heavy
+           with the stowed arm, and at the old gains the loaded legs lagged
+           their targets (d/p ~ 40 ms) until the body tipped, worst when
+           walking backwards. d kept at 20 (raising it adds tracking lag). -->
+      <xacro:pid_joint joint="front_left_hip_x"  p="900" i="12" d="20" i_min="-25" i_max="25"/>
+      <xacro:pid_joint joint="front_left_hip_y"  p="900" i="12" d="20" i_min="-25" i_max="25"/>
+      <xacro:pid_joint joint="front_left_knee"   p="900" i="12" d="20" i_min="-25" i_max="25"/>
+      <xacro:pid_joint joint="front_right_hip_x" p="900" i="12" d="20" i_min="-25" i_max="25"/>
+      <xacro:pid_joint joint="front_right_hip_y" p="900" i="12" d="20" i_min="-25" i_max="25"/>
+      <xacro:pid_joint joint="front_right_knee"  p="900" i="12" d="20" i_min="-25" i_max="25"/>
+      <xacro:pid_joint joint="rear_left_hip_x"   p="900" i="12" d="20" i_min="-25" i_max="25"/>
+      <xacro:pid_joint joint="rear_left_hip_y"   p="900" i="12" d="20" i_min="-25" i_max="25"/>
+      <xacro:pid_joint joint="rear_left_knee"    p="900" i="12" d="20" i_min="-25" i_max="25"/>
+      <xacro:pid_joint joint="rear_right_hip_x"  p="900" i="12" d="20" i_min="-25" i_max="25"/>
+      <xacro:pid_joint joint="rear_right_hip_y"  p="900" i="12" d="20" i_min="-25" i_max="25"/>
+      <xacro:pid_joint joint="rear_right_knee"   p="900" i="12" d="20" i_min="-25" i_max="25"/>
       <!-- Arm joints — arm0_shoulder_roll is fixed and excluded.
            init values = STOW_CONFIG from sim_manipulation_driver.py, so the

Commit message: debugging model from tipping over during RTF fluctuations

File: spot_description_sim/sdf/model.sdf.xacro (robot description, xacro)
@@ -63,5 +63,5 @@
           <ode>
             <kp>1e+07</kp>
-            <kd>100</kd>
+            <kd>1000</kd>
           </ode>
         </contact>
@@ -1070,5 +1070,8 @@
       name="ignition::gazebo::systems::JointStatePublisher">
       <topic>model/spot/joint_state</topic>
-      <update_rate>200</update_rate>
+      <!-- 100 Hz (was 200): halves bridge/TF wall-clock load so the sim-time
+           pipeline keeps up at higher RTF. Keep in sync with the controller
+           loop_rate and RSP publish_frequency (spot.gazebo.launch.py). -->
+      <update_rate>100</update_rate>
       <!-- Publish ONLY actuated joints, matching hardware
            /spot_driver/joint_states. Without this list the plugin publishes
@@ -1099,8 +1102,9 @@
       filename="ignition-gazebo-odometry-publisher-system"
       name="ignition::gazebo::systems::OdometryPublisher">
-      <!-- 100 Hz (was 10): at 10 Hz the odom stream was 20x sparser than the
-           200 Hz joint states, so TF odom->base updated in visible steps
-           relative to joint motion and EKF odom0 measurements were stale. -->
-      <odom_publish_frequency>100</odom_publish_frequency>
+      <!-- 50 Hz (was 100, originally 10): at 10 Hz the odom stream was far
+           sparser than the joint states, so TF odom->base updated in visible
+           steps and EKF odom0 measurements were stale. 50 Hz still oversamples
+           the 30 Hz footprint_to_odom EKF while halving bridge load. -->
+      <odom_publish_frequency>50</odom_publish_frequency>
       <odom_topic>/model/spot/odometry</odom_topic>
       <odom_frame>odom</odom_frame>
@@ -1121,21 +1125,25 @@
       name="ignition::gazebo::systems::JointTrajectoryController">
       <topic>model/spot/joint_trajectory</topic>
-      <!-- Leg gains: p raised 500->900 and i 1->12 (clamp widened to +/-25 Nm)
-           so stance legs stop sagging under load — the robot is rear-heavy
-           with the stowed arm, and at the old gains the loaded legs lagged
-           their targets (d/p ~ 40 ms) until the body tipped, worst when
-           walking backwards. d kept at 20 (raising it adds tracking lag). -->
-      <xacro:pid_joint joint="front_left_hip_x"  p="900" i="12" d="20" i_min="-25" i_max="25"/>
-      <xacro:pid_joint joint="front_left_hip_y"  p="900" i="12" d="20" i_min="-25" i_max="25"/>
-      <xacro:pid_joint joint="front_left_knee"   p="900" i="12" d="20" i_min="-25" i_max="25"/>
-      <xacro:pid_joint joint="front_right_hip_x" p="900" i="12" d="20" i_min="-25" i_max="25"/>
-      <xacro:pid_joint joint="front_right_hip_y" p="900" i="12" d="20" i_min="-25" i_max="25"/>
-      <xacro:pid_joint joint="front_right_knee"  p="900" i="12" d="20" i_min="-25" i_max="25"/>
-      <xacro:pid_joint joint="rear_left_hip_x"   p="900" i="12" d="20" i_min="-25" i_max="25"/>
-      <xacro:pid_joint joint="rear_left_hip_y"   p="900" i="12" d="20" i_min="-25" i_max="25"/>
-      <xacro:pid_joint joint="rear_left_knee"    p="900" i="12" d="20" i_min="-25" i_max="25"/>
-      <xacro:pid_joint joint="rear_right_hip_x"  p="900" i="12" d="20" i_min="-25" i_max="25"/>
-      <xacro:pid_joint joint="rear_right_hip_y"  p="900" i="12" d="20" i_min="-25" i_max="25"/>
-      <xacro:pid_joint joint="rear_right_knee"   p="900" i="12" d="20" i_min="-25" i_max="25"/>
+      <!-- Leg gains: aligned to the proven original CHAMP config (500/1/20,
+           PD-like — see champ_orig), with p scaled ~20% to 600 for the added
+           arm + RL kit payload so stance stiffness-to-weight matches the
+           original. i=1 with a tight ±1 Nm clamp (original used the plugin
+           default clamp): integral action wound up while a leg was unloaded
+           in swing and kicked at touchdown — the earlier 900/12/±25 gains
+           saturated the 80 Nm effort cap and caused twitch/stutter. d kept
+           at 20 (raising it adds tracking lag). If stance legs sag, raise p
+           toward 650 — do not raise i. -->
+      <xacro:pid_joint joint="front_left_hip_x"  p="600" i="1" d="20" i_min="-1" i_max="1"/>
+      <xacro:pid_joint joint="front_left_hip_y"  p="600" i="1" d="20" i_min="-1" i_max="1"/>
+      <xacro:pid_joint joint="front_left_knee"   p="600" i="1" d="20" i_min="-1" i_max="1"/>
+      <xacro:pid_joint joint="front_right_hip_x" p="600" i="1" d="20" i_min="-1" i_max="1"/>
+      <xacro:pid_joint joint="front_right_hip_y" p="600" i="1" d="20" i_min="-1" i_max="1"/>
+      <xacro:pid_joint joint="front_right_knee"  p="600" i="1" d="20" i_min="-1" i_max="1"/>
+      <xacro:pid_joint joint="rear_left_hip_x"   p="600" i="1" d="20" i_min="-1" i_max="1"/>
+      <xacro:pid_joint joint="rear_left_hip_y"   p="600" i="1" d="20" i_min="-1" i_max="1"/>
+      <xacro:pid_joint joint="rear_left_knee"    p="600" i="1" d="20" i_min="-1" i_max="1"/>
+      <xacro:pid_joint joint="rear_right_hip_x"  p="600" i="1" d="20" i_min="-1" i_max="1"/>
+      <xacro:pid_joint joint="rear_right_hip_y"  p="600" i="1" d="20" i_min="-1" i_max="1"/>
+      <xacro:pid_joint joint="rear_right_knee"   p="600" i="1" d="20" i_min="-1" i_max="1"/>
       <!-- Arm joints — arm0_shoulder_roll is fixed and excluded.
            init values = STOW_CONFIG from sim_manipulation_driver.py, so the
